File: navrh03_finished_almost/navrh03.kicad_pcb (KiCad board)
At the start: 2 copper layers, 88 parts, among them J10 Conn_01x03_Pin, J10R1 Conn_01x03_Pin, J11 Conn_01x03_Pin, J11R1 Conn_01x03_Pin, J12 Conn_01x03_Pin, J12R1 Conn_01x03_Pin, J13 Conn_01x03_Pin, J13R1 Conn_01x03_Pin, J14 Conn_01x03_Pin, J14R1 Conn_01x03_Pin, J15 Conn_01x03_Pin, J15R1 Conn_01x03_Pin, J16 Conn_01x03_Pin, J16R1 Conn_01x03_Pin, J17 Conn_01x03_Pin, J17R1 Conn_01x03_Pin, J18 Conn_01x03_Pin, J19 Conn_01x03_Pin, J2 Screw_Terminal_01x02, J20 Conn_01x03_Pin, J21 Conn_01x03_Pin, J22 Conn_01x03_Pin, J23 Conn_01x03_Pin, J24 Conn_01x03_Pin, J25 Conn_01x03_Pin, J26 Conn_01x03_Pin, J27 Conn_01x03_Pin, J28 Conn_01x11_Pin, J3 Conn_01x19_Pin, J4 Conn_01x03_Pin, J5 Conn_01x03_Pin, J6 Conn_01x03_Pin, J7 Conn_01x03_Pin, J8 Conn_01x03_Pin, J9 Conn_01x03_Pin, Q1 AOD417, U1-Left1 PCA9685, U2 PCA9685, U3 ESP32-DEVKITC-32UE

Commit message: Add files via upload
Parts:
- J28: footprint Connector_PinHeader_2.00mm:PinHeader_1x03_P2.00mm_Vertical -> Connector_PinHeader_2.00mm:PinHeader_1x11_P2.00mm_Vertical
- J3: footprint Connector_PinHeader_2.00mm:PinHeader_1x03_P2.00mm_Vertical -> Connector_PinHeader_2.00mm:PinHeader_1x19_P2.00mm_Vertical
- R7: value R -> RJP2
- R8J1: renamed from R8; value R -> RJP1
- moved J20 33.8 mm to (82.3, 73.7), turned to 90 degrees
- moved JP6 33.7 mm to (117.7, 65.8)
- moved JP1 33.7 mm to (117.7, 48.0)
- moved JP2 33.7 mm to (117.7, 51.3)
- moved JP3 33.7 mm to (117.7, 55.1)
- moved JP4 33.7 mm to (117.7, 58.7)
- moved JP5 33.7 mm to (117.7, 62.2)
- moved J3 33.2 mm to (167.6, 61.6)
- moved J21 30.5 mm to (82.3, 76.7), turned to 90 degrees
- moved J22 27.8 mm to (82.3, 79.8), turned to 90 degrees
- moved J19 26.0 mm to (124.9, 74.2), turned to -90 degrees
- moved J23 25.4 mm to (82.3, 82.8), turned to 90 degrees
- moved J10R1 24.6 mm to (176.3, 72.1), turned to 90 degrees
- moved J24 23.9 mm to (82.3, 85.9), turned to 90 degrees
- moved J11 23.9 mm to (210.2, 73.2), turned to -90 degrees
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Routing:
- net A5: track 399.6 -> 66.7 mm, vias 0 -> 6
- net GND: track 708.5 -> 447.7 mm, vias 0 -> 8
- net A2: track 20.2 -> 150.5 mm, vias 0 -> 6
- net A3: track 20.5 -> 148.8 mm, vias 0 -> 8
- net A1: track 20.1 -> 140.8 mm, vias 0 -> 6
- net A0: track 20.2 -> 133.1 mm, vias 0 -> 2
- net 5.0V: track 393.4 -> 327.0 mm, vias 0 -> 2
- net Net-(J3-Pin_10): track 0.00 -> 53.4 mm, vias 0 -> 2
- net Net-(J24-Pin_3): track 63.5 -> 11.4 mm
- net Net-(J3-Pin_11): track 0.00 -> 48.0 mm, vias 0 -> 2
- net Net-(J28-Pin_7): track 0.00 -> 47.8 mm, vias 0 -> 2
- net SCL0: track 80.4 -> 33.3 mm, vias 0 -> 2
- net Net-(J28-Pin_10): track 0.00 -> 47.0 mm, vias 0 -> 3
- net Net-(J23-Pin_3): track 57.1 -> 10.8 mm
- net Net-(J3-Pin_1): track 3.87 -> 46.8 mm, vias 0 -> 2
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