File: navrhAktualni/navrh03.kicad_pcb (KiCad board)
At the start: 2 copper layers, 88 parts, among them J10 Conn_01x03_Pin, J10R1 Conn_01x03_Pin, J11 Conn_01x03_Pin, J11R1 Conn_01x03_Pin, J12 Conn_01x03_Pin, J12R1 Conn_01x03_Pin, J13 Conn_01x03_Pin, J13R1 Conn_01x03_Pin, J14 Conn_01x03_Pin, J14R1 Conn_01x03_Pin, J15 Conn_01x03_Pin, J15R1 Conn_01x03_Pin, J16 Conn_01x03_Pin, J16R1 Conn_01x03_Pin, J17 Conn_01x03_Pin, J17R1 Conn_01x03_Pin, J18 Conn_01x03_Pin, J19 Conn_01x03_Pin, J2 Screw_Terminal_01x02, J20 Conn_01x03_Pin, J21 Conn_01x03_Pin, J22 Conn_01x03_Pin, J23 Conn_01x03_Pin, J24 Conn_01x03_Pin, J25 Conn_01x03_Pin, J26 Conn_01x03_Pin, J27 Conn_01x03_Pin, J28 Conn_01x11_Pin, J3 Conn_01x19_Pin, J4 Conn_01x03_Pin, J5 Conn_01x03_Pin, J6 Conn_01x03_Pin, J7 Conn_01x03_Pin, J8 Conn_01x03_Pin, J9 Conn_01x03_Pin, Q1 AOD417, U1-Left1 PCA9685, U2 PCA9685, U3 ESP32-DEVKITC-32UE

Commit message: NavrhMP check
Other:
- board outline added: 134.6 x 90.4 mm
Changed lines of the file:
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@@
 			(outputformat 1)
 			(mirror no)
-			(drillshape 1)
+			(drillshape 0)
 			(scaleselection 1)
 			(outputdirectory "")
@@
 		)
 	)
+	(gr_rect
+		(start 78.74 39.624)
+		(end 213.36 130.048)
+		(stroke
+			(width 0.05)
+			(type default)
+		)
+		(fill none)
+		(layer "Edge.Cuts")
+	)
 	(segment
 		(start 122.93 65.56)
@@
 		(start 146.304 117.364)
 		(end 166.608 117.364)
-		(width 0.2)
+		(width 0.5)
 		(layer "B.Cu")
 		(net 1)

Commit message: Add files via upload
Routing:
- net SCL1: track 76.2 -> 79.1 mm
- net GND: track 510.9 -> 512.8 mm
Changed lines of the file:
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@@
 		)
 		(property "Value" "Screw_Terminal_01x02"
-			(at 0 4.06 0)
+			(at -5.588 5.064 0)
 			(layer "F.Fab")
 			(effects
@@
 			(at 0 6.06 90)
 			(layer "F.Fab")
+			(hide yes)
 			(effects
 				(font
@@
 			(at 0 6.06 90)
 			(layer "F.Fab")
+			(hide yes)
 			(effects
 				(font
@@
 			(at 0 6.06 90)
 			(layer "F.Fab")
+			(hide yes)
 			(effects
 				(font
@@
 			(at 0 6.06 90)
 			(layer "F.Fab")
+			(hide yes)
 			(effects
 				(font
@@
 			(at 0 6.06 90)
 			(layer "F.Fab")
+			(hide yes)
 			(effects
 				(font
@@
 			(at 0 6.06 90)
 			(layer "F.Fab")
+			(hide yes)
 			(effects
 				(font
@@
 			(at 0 6.06 90)
 			(layer "F.Fab")
+			(hide yes)
 			(effects
 				(font
@@
 			(at 0 6.06 90)
 			(layer "F.Fab")
+			(hide yes)
 			(effects
 				(font
@@
 			(at 0 6.06 90)
 			(layer "F.Fab")
+			(hide yes)
 			(effects
 				(font
@@
 			(at 0 6.06 90)
 			(layer "F.Fab")
+			(hide yes)
 			(effects
 				(font
@@
 			(at 0 6.06 90)
 			(layer "F.Fab")
+			(hide yes)
 			(effects
 				(font
@@
 			(at 0 6.06 90)
 			(layer "F.Fab")
+			(hide yes)
 			(effects
 				(font
@@
 			(at 0 6.06 90)
 			(layer "F.Fab")
+			(hide yes)
 			(effects
 				(font
@@
 			(at 0 6.06 90)
 			(layer "F.Fab")
+			(hide yes)
 			(effects
 				(font
@@
 		)
 		(property "Value" "AOD417"
-			(at -4.0066 7.7668 0)
+			(at -2.54 11.684 0)
 			(unlocked yes)
 			(layer "F.Fab")
@@
 		)
 		(property "Value" "PCA9685"
-			(at 5.588 2.032 0)
+			(at -0.508 1.524 0)
 			(unlocked yes)
 			(layer "F.Fab")
@@
 			(at 0 6.06 90)
 			(layer "F.Fab")
+			(hide yes)
 			(effects
 				(font
@@
 	)
 	(segment
-		(start 175.796 93.92)
-		(end 175.796 100.556)
+		(start 176.244 93.472)
+		(end 176.244 100.108)
+		(width 0.5)
+		(layer "F.Cu")
+		(net 1)
+	)
+	(segment
+		(start 146.304 107.188)
+		(end 146.304 108.204)
 		(width 0.5)
 		(layer "F.Cu")
@@
 	)
 	(segment
-		(start 169.164 107.188)
-		(end 146.304 107.188)
-		(width 0.5)
-		(layer "F.Cu")
-		(net 1)
-	)
-	(segment
 		(start 124.968 98.552)
 		(end 124.968 98.044)
@@
 	)
 	(segment
-		(start 146.304 107.188)
-		(end 146.304 108.204)
-		(width 0.5)
-		(layer "F.Cu")
-		(net 1)
-	)
-	(segment
 		(start 190.5822 84.725)
 		(end 190.5822 85.7698)
@@
 	)
 	(segment
+		(start 176.244 100.108)
+		(end 169.164 107.188)
+		(width 0.5)
+		(layer "F.Cu")
+		(net 1)
+	)
+	(segment
 		(start 152.146 119.406)
 		(end 154.2275 121.4875)
@@
 	)
 	(segment
+		(start 169.164 107.188)
+		(end 146.304 107.188)
+		(width 0.5)
+		(layer "F.Cu")
+		(net 1)
+	)
+	(segment
 		(start 101.6 85.3748)
 		(end 101.2222 84.997)
@@
 	)
 	(segment
-		(start 176.244 93.472)
-		(end 175.796 93.92)
-		(width 0.5)
-		(layer "F.Cu")
-		(net 1)
-	)
-	(segment
 		(start 123.093 58.448)
 		(end 123.093 62.512)
@@
 	)
 	(segment
-		(start 175.796 100.556)
-		(end 169.164 107.188)
-		(width 0.5)
-		(layer "F.Cu")
-		(net 1)
-	)
-	(segment
 		(start 123.093 55.308)
 		(end 123.093 58.448)
@@
 	)
 	(segment
-		(start 210.248 73.152)
-		(end 208.596 71.5)
-		(width 0.2)
-		(layer "B.Cu")
-		(net 1)
-	)
-	(segment
 		(start 82.296 94.996)
 		(end 89.916 102.616)
@@
 	)
 	(segment
+		(start 204.344 71.5)
+		(end 200.5 75.344)
+		(width 0.2)
+		(layer "B.Cu")
+		(net 1)
+	)
+	(segment
 		(start 108.070756 78.497)
 		(end 102.616 83.951756)
@@
 	)
 	(segment
+		(start 210.248 72.072)
+		(end 209.676 71.5)
+		(width 0.2)
+		(layer "B.Cu")
+		(net 1)
+	)
+	(segment
 		(start 123.952 71.628)
 		(end 124.46 71.12)
@@
 	)
 	(segment
-		(start 208.596 71.5)
-		(end 206.5 71.5)
-		(width 0.2)
-		(layer "B.Cu")
-		(net 1)
-	)
-	(segment
 		(start 132.08 106.68)
 		(end 142.764 117.364)
@@
 	)
 	(segment
-		(start 206.5 71.5)
-		(end 200.5 77.5)
+		(start 210.248 73.152)
+		(end 210.248 72.072)
 		(width 0.2)
 		(layer "B.Cu")
@@
 	)
 	(segment
+		(start 200.5 75.344)
+		(end 200.5 77.5)
+		(width 0.2)
+		(layer "B.Cu")
+		(net 1)
+	)
+	(segment
 		(start 210.28 95.363)
 		(end 210.28 94.488)
-		(width 0.2)
+		(width 0.5)
 		(layer "B.Cu")
 		(net 1)
@@
 	)
 	(segment
+		(start 209.676 71.5)
+		(end 204.344 71.5)
+		(width 0.2)
+		(layer "B.Cu")
+		(net 1)
+	)
+	(segment
 		(start 178.276 72.136)
 		(end 178.276 71.152)
@@
 	(segment
 		(start 99.06 79.756)
-		(end 99.06 79.556001)
-		(width 0.2)
-		(layer "F.Cu")
-		(net 73)
-	)
-	(segment
-		(start 99.06 79.756)
 		(end 101.1812 79.756)
 		(width 0.2)
@@
 	)
 	(segment
-		(start 97.668 80.971999)
-		(end 97.668 80.772)
-		(width 0.2)
-		(layer "F.Cu")
-		(net 74)
-	)
-	(segment
 		(start 97.668 80.772)
 		(end 98.143314 80.772)
@@
 	)
 	(segment
-		(start 135.292244 71.48)
-		(end 163.939067 71.48)
+		(start 134.352244 70.54)
+		(end 135.292244 71.48)
 		(width 0.2)
 		(layer "B.Cu")
@@
 	)
 	(segment
-		(start 133.871756 70.54)
-		(end 134.352244 70.54)
+		(start 133.532 70.879756)
+		(end 133.871756 70.54)
+		(width 0.2)
+		(layer "B.Cu")
+		(net 89)
+	)
+	(segment
+		(start 164.56 73.988574)
+		(end 167.244426 76.673)
 		(width 0.2)
 		(layer "B.Cu")
@@
 	)
 	(segment
-		(start 135.636 73.66)
-		(end 133.532 71.556)
+		(start 135.292244 71.48)
+		(end 163.939067 71.48)
 		(width 0.2)
 		(layer "B.Cu")
@@
 	)
 	(segment
-		(start 197.069 76.673)
-		(end 197.640536 77.244536)
+		(start 197.612 76.067756)
+		(end 197.42 76.259756)
 		(width 0.2)
 		(layer "B.Cu")
@@
 	(segment
 		(start 167.244426 76.673)
-		(end 197.069 76.673)
+		(end 183.628244 76.673)
 		(width 0.2)
 		(layer "B.Cu")
@@
 	)
 	(segment
-		(start 134.352244 70.54)
-		(end 135.292244 71.48)
+		(start 133.871756 70.54)
+		(end 134.352244 70.54)
 		(width 0.2)
 		(layer "B.Cu")
@@
 	)
 	(segment
-		(start 133.532 70.879756)
-		(end 133.871756 70.54)
+		(start 183.968 76.333244)
+		(end 183.968 75.852756)
 		(width 0.2)
 		(layer "B.Cu")
@@
 	)
 	(segment
-		(start 164.56 73.988574)
-		(end 167.244426 76.673)
+		(start 197.612 75.184)
+		(end 197.612 76.067756)
+		(width 0.2)
+		(layer "B.Cu")
+		(net 89)
+	)
+	(segment
+		(start 197.42 77.024)
+		(end 197.640536 77.244536)
+		(width 0.2)
+		(layer "B.Cu")
+		(net 89)
+	)
+	(segment
+		(start 183.628244 76.673)
+		(end 183.968 76.333244)
+		(width 0.2)
+		(layer "B.Cu")
+		(net 89)
+	)
+	(segment
+		(start 183.968 75.852756)
+		(end 184.636756 75.184)
+		(width 0.2)
+		(layer "B.Cu")
+		(net 89)
+	)
+	(segment
+		(start 184.636756 75.184)
+		(end 197.612 75.184)
+		(width 0.2)
+		(layer "B.Cu")
+		(net 89)
+	)
+	(segment
+		(start 197.42 76.259756)
+		(end 197.42 77.024)
 		(width 0.2)
 		(layer "B.Cu")
@@
 	)
 	(segment
+		(start 135.636 73.66)
+		(end 133.532 71.556)
+		(width 0.2)
+		(layer "B.Cu")
+		(net 89)
+	)
+	(segment
 		(start 165.608 63.5)
 		(end 164.62 63.5)
@@
 	)
 	(segment
-		(start 135.232 57.3)
+		(start 135.74 57.3)
+		(end 131.064 61.976)
+		(width 0.2)
+		(layer "F.Cu")
+		(net 108)
+	)
+	(segment
+		(start 131.064 61.976)
 		(end 130.556 61.976)
 		(width 0.2)
@@
 	(segment
 		(start 138.1 57.3)
-		(end 135.232 57.3)
+		(end 135.74 57.3)
 		(width 0.2)
 		(layer "F.Cu")
